File: MCP73834_li-ion charger.sch (KiCad schematic (older format))
At the start: 15 parts

Commit message: associated components
Parts:
- removed U?: MCP73834-FCI/UN, symbol MCP73834-FCI/UN
- added CON101: USB-MICRO-B, Connect:USB_Micro-B, symbol USB-MICRO-B
- added P102: CONN_01X06, Pin_Headers:Pin_Header_Straight_1x06, symbol CONN_01X06
- added P104: CONN_01X02, Pin_Headers:Pin_Header_Straight_1x02, symbol CONN_01X02
- added U101: MCP73834-FCI/UN, Housings_SSOP:MSOP-10-1EP_3x3mm_Pitch0.5mm, symbol MCP73834-FCI/UN
- C101: renamed from C?; value C -> 1 uF; footprint (none) -> Capacitors_SMD:C_0805_HandSoldering
- C102: renamed from C?; value C -> 4.7 uF; footprint (none) -> Capacitors_SMD:C_0805_HandSoldering
- D101, D102, D103: renamed from D?; footprint (none) -> LEDs:LED-0805
- P101: renamed from P?; footprint (none) -> Pin_Headers:Pin_Header_Straight_1x02
- P103: renamed from P?; footprint (none) -> battery logger:Terminal_Block_1x2_3.5mm
- R101, R102, R103: renamed from R?; value R -> 470R; footprint (none) -> Resistors_SMD:R_0805_HandSoldering
- R104: renamed from R?; value R -> 1k; footprint (none) -> Resistors_SMD:R_0805_HandSoldering
- R105, R106: renamed from R?; footprint (none) -> Resistors_SMD:R_0805_HandSoldering
- TH101: renamed from TH?; footprint (none) -> battery logger:SolderWirePad_2x_0-8mmDrill
Connections:
- net labels added: Prog
- wire segments 50 -> 60
- no-connect marks 0 -> 3
Other:
- moved on the sheet: C101, C102, D101, D102, D103, P101, P103, R101, R102, R103, R104, R105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

Commit message: started layout
Parts:
- removed P101: CONN_01X02, Pin_Headers:Pin_Header_Straight_1x02, symbol CONN_01X02
- CON101: footprint Connect:USB_Micro-B -> USB connectors:USB_Micro-B_FCI_10118193-0001LF; MPN (none) -> 10118193-0001LF
- TH101: footprint battery logger:SolderWirePad_2x_0-8mmDrill -> Pin_Headers:Pin_Header_Straight_1x02
Connections:
- wire segments 60 -> 56
Changed lines of the file:
@@
 F 0 "TH101" V 7610 3515 50  0000 C CNN
 F 1 "THERMISTOR" V 7410 3465 50  0000 C BNN
-F 2 "battery logger:SolderWirePad_2x_0-8mmDrill" H 7510 3465 60  0001 C CNN
+F 2 "Pin_Headers:Pin_Header_Straight_1x02" H 7510 3465 60  0001 C CNN
 F 3 "" H 7510 3465 60  0000 C CNN
 	1    7510 3465
@@
 	1    8750 2955
 	1    0    0    -1
-$EndComp
-$Comp
-L CONN_01X02 P101
-U 1 1 551584CA
-P 2910 1480
-F 0 "P101" H 2910 1630 50  0000 C CNN
-F 1 "CONN_01X02" V 3010 1480 50  0000 C CNN
-F 2 "Pin_Headers:Pin_Header_Straight_1x02" H 2910 1480 60  0001 C CNN
-F 3 "" H 2910 1480 60  0000 C CNN
-	1    2910 1480
-	-1   0    0    -1
 $EndComp
 $Comp
@@
 $Comp
 L GND #PWR03
-U 1 1 5515F1E2
-P 3135 1580
-F 0 "#PWR03" H 3135 1330 60  0001 C CNN
-F 1 "GND" H 3135 1430 60  0001 C CNN
-F 2 "" H 3135 1580 60  0000 C CNN
-F 3 "" H 3135 1580 60  0000 C CNN
-F 4 "Value" H 3135 1580 60  0001 C CNN "MPN"
-	1    3135 1580
-	1    0    0    -1
-$EndComp
-$Comp
-L GND #PWR04
 U 1 1 5515F7C0
 P 3850 2590
-F 0 "#PWR04" H 3850 2340 60  0001 C CNN
+F 0 "#PWR03" H 3850 2340 60  0001 C CNN
 F 1 "GND" H 3850 2440 60  0001 C CNN
 F 2 "" H 3850 2590 60  0000 C CNN
@@
 $EndComp
 $Comp
-L GND #PWR05
+L GND #PWR04
 U 1 1 5515F86B
 P 3165 2585
-F 0 "#PWR05" H 3165 2335 60  0001 C CNN
+F 0 "#PWR04" H 3165 2335 60  0001 C CNN
 F 1 "GND" H 3165 2435 60  0001 C CNN
 F 2 "" H 3165 2585 60  0000 C CNN
@@
 $EndComp
 $Comp
-L GND #PWR06
+L GND #PWR05
 U 1 1 551608B7
 P 8550 3060
-F 0 "#PWR06" H 8550 2810 60  0001 C CNN
+F 0 "#PWR05" H 8550 2810 60  0001 C CNN
 F 1 "GND" H 8550 2910 60  0001 C CNN
 F 2 "" H 8550 3060 60  0000 C CNN
@@
 $EndComp
 $Comp
-L GND #PWR07
+L GND #PWR06
 U 1 1 55160A39
 P 8550 3500
-F 0 "#PWR07" H 8550 3250 60  0001 C CNN
+F 0 "#PWR06" H 8550 3250 60  0001 C CNN
 F 1 "GND" H 8550 3350 60  0001 C CNN
 F 2 "" H 8550 3500 60  0000 C CNN
@@
 Wire Wire Line
 	2705 4155 2705 4210
-Wire Wire Line
-	3110 1430 3300 1430
-Wire Wire Line
-	3300 1430 3300 1930
-Connection ~ 3300 1930
-Wire Wire Line
-	3110 1530 3135 1530
-Wire Wire Line
-	3135 1530 3135 1580
 Wire Wire Line
 	3850 2500 3850 2590
@@
 F 0 "CON101" H 2270 2480 50  0000 C CNN
 F 1 "USB-MICRO-B" H 2420 1780 50  0000 C CNN
-F 2 "Connect:USB_Micro-B" H 2570 2030 50  0001 C CNN
-F 3 "" H 2570 2030 50  0000 C CNN
+F 2 "USB connectors:USB_Micro-B_FCI_10118193-0001LF" H 2570 2030 50  0001 C CNN
+F 3 "http://portal.fciconnect.com/Comergent//fci/drawing/10118193.pdf" H 2570 2030 50  0001 C CNN
+F 4 "10118193-0001LF" H 2570 2130 60  0001 C CNN "MPN"
 	1    2570 2130
 	-1   0    0    -1
