File: $MCP73834_li-ion charger.sch (KiCad schematic (older format))
At the start: 17 parts, among them CON101 USB-MICRO-B, P102 CONN_01X06, P103 CONN_01X02, P104 CONN_01X02, U101 MCP73834-FCI/UN

Commit message: finished layout
Connections:
- net labels added: Th
Changed lines of the file:
@@
 Text Label 3190 1930 0    28   ~ 0
 Vs
+Text Label 6340 3105 0    28   ~ 0
+Th
 $EndSCHEMATC
